File: NewRemote/BasePlate.brd (EAGLE design)
At the start: 186 x 120 mm, 7 parts

Commit message: A bunch of new parts
Parts:
- moved E$5 1.00 mm to (-40.0, -53.0)
Other:
- board size 186 x 120 mm -> 292.2 x 120 mm
Changed lines of the file:
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@@
 <board>
 <plain>
-<wire x1="-93" y1="60" x2="-33" y2="60" width="0.254" layer="20"/>
-<wire x1="-33" y1="60" x2="-28" y2="55" width="0.254" layer="20" curve="-90"/>
-<wire x1="-28" y1="55" x2="-28" y2="-6" width="0.254" layer="20"/>
-<wire x1="-28" y1="-6" x2="-23" y2="-11" width="0.254" layer="20" curve="90"/>
-<wire x1="-23" y1="-11" x2="25" y2="-11" width="0.254" layer="20"/>
-<wire x1="25" y1="-11" x2="30" y2="-6" width="0.254" layer="20" curve="90"/>
-<wire x1="30" y1="-6" x2="30" y2="55" width="0.254" layer="20"/>
-<wire x1="30" y1="55" x2="35" y2="60" width="0.254" layer="20" curve="-90"/>
-<wire x1="35" y1="60" x2="93" y2="60" width="0.254" layer="20"/>
-<wire x1="93" y1="-60" x2="-93" y2="-60" width="0.254" layer="20"/>
-<dimension x1="-93" y1="60" x2="-87" y2="-60" x3="-156" y3="0" textsize="1.778" layer="47" dtype="vertical" unit="inch"/>
-<wire x1="-93" y1="60" x2="-146" y2="0" width="0.254" layer="47" curve="90"/>
-<wire x1="-146" y1="0" x2="-93" y2="-60" width="0.254" layer="47" curve="90"/>
-<wire x1="93" y1="-60" x2="146" y2="0" width="0.254" layer="47" curve="90"/>
-<wire x1="146" y1="0" x2="93" y2="60" width="0.254" layer="47" curve="90"/>
-<dimension x1="-146" y1="0" x2="146" y2="0" x3="0" y3="87" textsize="1.778" layer="47" dtype="horizontal" unit="inch"/>
+<wire x1="-93" y1="60" x2="-33" y2="60" width="0.0254" layer="20"/>
+<wire x1="-33" y1="60" x2="-28" y2="55" width="0.0254" layer="20" curve="-90"/>
+<wire x1="-28" y1="55" x2="-28" y2="-6" width="0.0254" layer="20"/>
+<wire x1="-28" y1="-6" x2="-23" y2="-11" width="0.0254" layer="20" curve="90"/>
+<wire x1="-23" y1="-11" x2="25" y2="-11" width="0.0254" layer="20"/>
+<wire x1="25" y1="-11" x2="30" y2="-6" width="0.0254" layer="20" curve="90"/>
+<wire x1="30" y1="-6" x2="30" y2="55" width="0.0254" layer="20"/>
+<wire x1="30" y1="55" x2="35" y2="60" width="0.0254" layer="20" curve="-90"/>
+<wire x1="35" y1="60" x2="93" y2="60" width="0.0254" layer="20"/>
+<wire x1="93" y1="-60" x2="-93" y2="-60" width="0.0254" layer="20"/>
+<dimension x1="-93" y1="60" x2="-87" y2="-60" x3="-148" y3="0" textsize="1.778" layer="47" dtype="vertical" unit="inch"/>
+<wire x1="-93" y1="60" x2="-146" y2="0" width="0.0254" layer="20" curve="90"/>
+<wire x1="-146" y1="0" x2="-93" y2="-60" width="0.0254" layer="20" curve="90"/>
+<wire x1="93" y1="-60" x2="146" y2="0" width="0.0254" layer="20" curve="90"/>
+<wire x1="146" y1="0" x2="93" y2="60" width="0.0254" layer="20" curve="90"/>
+<dimension x1="-146" y1="0" x2="146" y2="0" x3="0" y3="61" textsize="1.778" layer="47" dtype="horizontal" unit="inch"/>
+<wire x1="-90" y1="19" x2="-78" y2="19" width="0.0254" layer="20"/>
+<wire x1="-78" y1="19" x2="-76" y2="17" width="0.0254" layer="20" curve="-90"/>
+<wire x1="-76" y1="17" x2="-76" y2="-17" width="0.0254" layer="20"/>
+<wire x1="-76" y1="-17" x2="-78" y2="-19" width="0.0254" layer="20" curve="-90"/>
+<wire x1="-78" y1="-19" x2="-90" y2="-19" width="0.0254" layer="20"/>
+<wire x1="-90" y1="-19" x2="-92" y2="-21" width="0.0254" layer="20" curve="90"/>
+<wire x1="-92" y1="-21" x2="-92" y2="-23" width="0.0254" layer="20"/>
+<wire x1="-92" y1="25" x2="-92" y2="21" width="0.0254" layer="20"/>
+<wire x1="-92" y1="21" x2="-90" y2="19" width="0.0254" layer="20" curve="90"/>
+<wire x1="-92" y1="25" x2="-94" y2="27" width="0.0254" layer="20" curve="90"/>
+<wire x1="-94" y1="27" x2="-130" y2="27" width="0.0254" layer="20"/>
+<wire x1="-130" y1="27" x2="-132" y2="25" width="0.0254" layer="20" curve="90"/>
+<wire x1="-132" y1="25" x2="-132" y2="21" width="0.0254" layer="20"/>
+<wire x1="-132" y1="21" x2="-134" y2="19" width="0.0254" layer="20" curve="-90"/>
+<wire x1="-134" y1="19" x2="-135" y2="19" width="0.0254" layer="20"/>
+<wire x1="-135" y1="-19" x2="-134" y2="-19" width="0.0254" layer="20"/>
+<wire x1="-134" y1="-19" x2="-132" y2="-21" width="0.0254" layer="20" curve="-90"/>
+<wire x1="-132" y1="-21" x2="-132" y2="-23" width="0.0254" layer="20"/>
+<wire x1="-132" y1="-23" x2="-130" y2="-25" width="0.0254" layer="20" curve="90"/>
+<wire x1="-130" y1="-25" x2="-94" y2="-25" width="0.0254" layer="20"/>
+<wire x1="-94" y1="-25" x2="-92" y2="-23" width="0.0254" layer="20" curve="90"/>
+<wire x1="-135" y1="19" x2="-137" y2="17" width="0.0254" layer="20" curve="90"/>
+<wire x1="-137" y1="17" x2="-137" y2="-17" width="0.0254" layer="20"/>
+<wire x1="-137" y1="-17" x2="-135" y2="-19" width="0.0254" layer="20" curve="90"/>
+<wire x1="90" y1="-19" x2="77" y2="-19" width="0.0254" layer="20"/>
+<wire x1="77" y1="-19" x2="75" y2="-17" width="0.0254" layer="20" curve="-90"/>
+<wire x1="75" y1="-17" x2="75" y2="17" width="0.0254" layer="20"/>
+<wire x1="75" y1="17" x2="77" y2="19" width="0.0254" layer="20" curve="-90"/>
+<wire x1="77" y1="19" x2="90" y2="19" width="0.0254" layer="20"/>
+<wire x1="90" y1="19" x2="92" y2="21" width="0.0254" layer="20" curve="90"/>
+<wire x1="92" y1="21" x2="92" y2="23" width="0.0254" layer="20"/>
+<wire x1="92" y1="-25" x2="92" y2="-21" width="0.0254" layer="20"/>
+<wire x1="92" y1="-21" x2="90" y2="-19" width="0.0254" layer="20" curve="90"/>
+<wire x1="92" y1="-25" x2="94" y2="-27" width="0.0254" layer="20" curve="90"/>
+<wire x1="94" y1="-27" x2="130" y2="-27" width="0.0254" layer="20"/>
+<wire x1="130" y1="-27" x2="132" y2="-25" width="0.0254" layer="20" curve="90"/>
+<wire x1="132" y1="-25" x2="132" y2="-21" width="0.0254" layer="20"/>
+<wire x1="132" y1="-21" x2="134" y2="-19" width="0.0254" layer="20" curve="-90"/>
+<wire x1="134" y1="-19" x2="135" y2="-19" width="0.0254" layer="20"/>
+<wire x1="135" y1="19" x2="134" y2="19" width="0.0254" layer="20"/>
+<wire x1="134" y1="19" x2="132" y2="21" width="0.0254" layer="20" curve="-90"/>
+<wire x1="132" y1="21" x2="132" y2="23" width="0.0254" layer="20"/>
+<wire x1="132" y1="23" x2="130" y2="25" width="0.0254" layer="20" curve="90"/>
+<wire x1="130" y1="25" x2="94" y2="25" width="0.0254" layer="20"/>
+<wire x1="94" y1="25" x2="92" y2="23" width="0.0254" layer="20" curve="90"/>
+<wire x1="135" y1="-19" x2="137" y2="-17" width="0.0254" layer="20" curve="90"/>
+<wire x1="137" y1="-17" x2="137" y2="17" width="0.0254" layer="20"/>
+<wire x1="137" y1="17" x2="135" y2="19" width="0.0254" layer="20" curve="90"/>
 </plain>
 <attributes>
@@
 <element name="E$3" library="RemotePartsA" package="FRSKY-TARANIS-GIMBAL" value="" x="-108" y="0" locked="yes"/>
 <element name="E$4" library="RemotePartsA" package="FRSKY-TARANIS-GIMBAL" value="" x="108" y="0" locked="yes" rot="R180"/>
-<element name="E$5" library="RemotePartsA" package="SPARKFUN_LCD_33" value="" x="-39" y="-53" locked="yes"/>
+<element name="E$5" library="RemotePartsA" package="SPARKFUN_LCD_33" value="" x="-40" y="-53" locked="yes"/>
 <element name="E$6" library="RemotePartsA" package="CONTROLLER_OUTLINE" value="" x="0" y="0" locked="yes"/>
 <element name="E$7" library="BOBs" package="ATMEGA128RFA1" value="" x="-25.5" y="58.5" locked="yes" rot="R270"/>
