File: NewRemote/controller_board.brd (EAGLE design)
At the start: 144 x 118 mm, 34 parts, among them J1 FRSKY-GIMBAL, J2 FRSKY-GIMBAL, J3 WIRE-HARNESS-SPARKFUN-9915

Commit message: A bunch of new parts
Parts:
- removed BTN1: BUTTON-TACTILE-SQUARE, Controller:BUTTON-TACTILE-SQUARE-ADAFRUIT1010
- removed P-1, R-1, T-1, Y-1: JST_3PIN_GND_VDD_SIG, RemotePartsB:JST-3-PTH-REVERSE
- removed R1, R2: 10K, KoalaBuild:RESAD770W45L370D210_HS
- added 3.3V, GND, VBAT: (no value), Components:SCREW-TERMINAL-1X3-2.54MM
- added C1: (no value), KoalaBuild:CAPPRD750W80D1800H2200P
- added C2: (no value), KoalaBuild:CAPPRD250W80D630H1220P
- added D3: BLUE, Components:LED3MM
- added D4: RED, Components:LED3MM
- added D5: GREEN, Components:LED3MM
- added F1: SHORT, RemotePartsB:SHORT
- added J10, J8, J9: (no value), Components:HDRV3W63P254_3X1_762X254H838_HS
- added J12, J14, J16, J18: JST_3PIN_GND_VDD_SIG, RemotePartsB:JST-3-PTH-REVERSE
- added J6: HEADER-0.1IN-6POS-SCREW, Components:SCREW-TERMINAL-1X6-2.54MM
- added J7: HEADER-0.1IN-6POS-FEMALE, Components:HDRV6W63P254_6X1_1524X254H838_HS
- added R4, R5: (no value), KoalaBuild:RESAD770W45L370D210_HS
- added RESET: BUTTON-TACTILE-SQUARE, Controller:BUTTON-TACTILE-SQUARE-ADAFRUIT1010
- moved J3 36.4 mm to (-65.5, 19.5), turned to 180 degrees
- moved BATT4 16.0 mm to (-53.0, 11.5), flipped to the top
- moved BATT1 16.0 mm to (53.0, 11.0), flipped to the top
- moved U$3 13.1 mm to (-12.0, 17.0)
- moved BATT2 10.5 mm to (37.0, 16.5), flipped to the top
- moved BATT3 10.5 mm to (-37.0, 17.0), flipped to the top
- moved U$1 9.51 mm to (-16.5, 7.50)
- moved U$2 4.50 mm to (11.0, 20.0)
- moved D1 2.00 mm to (26.5, 0.00)
- moved LCD 1.00 mm to (-40.0, -53.0)
- moved TM1 1.00 mm to (23.0, -8.00)
- moved J4 0.17 mm to (16.0, 14.2)
- turned B1 to 0 degrees
- renumbered P-2 to J11, R-2 to J13, T-2 to J15, U$5 to S1, Y-2 to J17
Connections:
- removed net N$10: J5.2, U$4.PD6
- removed net N$11: J5.3, U$4.PD5
- removed net N$12: J5.4, U$4.PD4
- new net BATGND: BATT4.N1, BATT4.N2, C1.2, D1.K, F1.B, GND.1, GND.3, J10.1, J10.2, J10.3, J3.BLACK, S1.P$3, S1.P$6
- new net D18: J4.2, J6.5, J7.5, U$4.PG2
- new net D19: J4.1, J6.6, J7.6, U$4.PG5
- new net D3: J6.1, J7.1, U$4.J2.D3
- new net D4: J6.2, J7.2, U$4.PE4
- new net D5: J6.3, J7.3, U$4.J2.D5
- new net D9: J6.4, J7.4, U$4.J2.D9
- new net LED_BLUE: D3.A, J5.2, U$4.PD6
- new net LED_GREEN: D5.A, J5.3, U$4.PD5
- new net LED_RED: D4.A, J5.4, U$4.PD4
- net +3V3: now also 3.3V.1, 3.3V.2, 3.3V.3, C2.1, J12.2, J14.2, J16.2, J18.2, J8.1, J8.2, J8.3; no longer P-1.2, R-1.2, T-1.2, Y-1.2
- net BTN1: no longer R1.2
- net BTN2: no longer R2.2
- net GND: now also C2.2, D3.K, F1.A, J12.1, J14.1, J16.1, J18.1, R4.1, R5.1, RESET.S, RESET.S2, U$4.GND2; no longer BATT4.N1, BATT4.N2, BTN1.S, BTN1.S2, D1.K, J3.BLACK, P-1.1, R-1.1, R1.1, R2.1, S1.P$3, S1.P$6, T-1.1, Y-1.1
- net N$4: now also D4.K, R4.2; no longer J4.1, U$4.PG5
- net N$6: now also D5.K, R5.2; no longer J4.2, U$4.PG2
- net PITCH: now also J12.3; no longer P-1.3
- net RESET: now also RESET.P, RESET.P2; no longer BTN1.P, BTN1.P2
- net ROLL: now also J14.3; no longer R-1.3
- net THROTTLE: now also J16.3; no longer T-1.3
- net VBAT: now also C1.1, J9.1, J9.2, J9.3, VBAT.1, VBAT.2, VBAT.3
- net YAW: now also J18.3; no longer Y-1.3
Routing:
- net BATGND: track 0.00 -> 261.5 mm
- net LED_GREEN: track 0.00 -> 130.3 mm, vias 0 -> 3
- net LED_RED: track 0.00 -> 105.1 mm
- net LED_BLUE: track 0.00 -> 102.9 mm
- net D4: track 0.00 -> 86.5 mm, vias 0 -> 1
- net VBAT: track 135.8 -> 221.7 mm, vias 0 -> 3
- net D3: track 0.00 -> 77.8 mm
- net D18: track 0.00 -> 74.3 mm
- net D5: track 0.00 -> 71.7 mm
- net D19: track 0.00 -> 65.4 mm
- net D9: track 0.00 -> 62.1 mm
- net +3V3: track 442.9 -> 497.1 mm, vias 0 -> 1
- net TX1: track 75.6 -> 114.3 mm, vias 1 -> 0
- net BTN1: track 121.8 -> 142.9 mm
- net RESET: track 25.5 -> 42.9 mm
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Other:
- outline, holes or cut-outs redrawn
- board text added: "PITCH"
- board text added: "ROLL"
- board text added: "THR"
- board text added: "YAW"
- board text removed: "RESET"
