File: NewRemote/controller_board.sch (EAGLE design)
At the start: 30 parts, among them J1 FRSKY-GIMBAL, J2 FRSKY-GIMBAL, J3 WIRE-HARNESS-SPARKFUN-9915

Commit message: A bunch of new parts
Parts:
- removed R1, R2: 10K, KoalaBuild:RESOLVED-RESISTOR_TH-1/6W-CARBON
- added 3.3V, GND, VBAT: (no value), Components:HEADER-0.1IN-3POS-SCREW
- added C1: (no value), KoalaBuild:RESOLVED-CAPACITOR-POL_TH-RADIAL_ALUMINUM_18MM
- added C2: (no value), KoalaBuild:RESOLVED-CAPACITOR-POL_TH-RADIAL_ALUMINUM_6.3MM
- added D3: BLUE, Components:LED3MM
- added D4: RED, Components:LED3MM
- added D5: GREEN, Components:LED3MM
- added F1: SHORT, RemotePartsB:SHORT
- added J10, J8, J9: (no value), Components:HEADER-0.1IN-3POS-FEMALE
- added J6: HEADER-0.1IN-6POS-SCREW, Components:HEADER-0.1IN-6POS-SCREW
- added J7: HEADER-0.1IN-6POS-FEMALE, Components:HEADER-0.1IN-6POS-FEMALE
- added R4, R5: (no value), KoalaBuild:RESOLVED-RESISTOR_TH-1/6W-CARBON
- renumbered BTN1 to RESET, P-1 to J12, P-2 to J11, R-1 to J14, R-2 to J13, T-1 to J16, T-2 to J15, U$5 to S1, Y-1 to J18, Y-2 to J17
Connections:
- removed net N$10: J5.2, U$4.PD6
- removed net N$11: J5.3, U$4.PD5
- removed net N$12: J5.4, U$4.PD4
- new net BATGND: BATT4.N, C1.-, D1.C, F1.B, GND.1, GND.3, J10.1, J10.2, J10.3, J3.BLACK, S1.OFF
- new net D18: J4.2, J6.5, J7.5, U$4.PG2
- new net D19: J4.1, J6.6, J7.6, U$4.PG5
- new net D3: J6.1, J7.1, U$4.D3~
- new net D4: J6.2, J7.2, U$4.PE4~
- new net D5: J6.3, J7.3, U$4.D5~
- new net D9: J6.4, J7.4, U$4.D9~
- new net LED_BLUE: D3.A, J5.2, U$4.PD6
- new net LED_GREEN: D5.A, J5.3, U$4.PD5
- new net LED_RED: D4.A, J5.4, U$4.PD4
- net +3V3: now also 3.3V.1, 3.3V.2, 3.3V.3, C2.+, J8.1, J8.2, J8.3
- net BTN1: no longer R1.2
- net BTN2: no longer R2.2
- net GND: now also C2.-, D3.C, F1.A, R4.1, R5.1; no longer BATT4.N, D1.C, J3.BLACK, R1.1, R2.1, S1.OFF, U$4.GND1
- net N$4: now also D4.C, R4.2; no longer J4.1, U$4.PG5
- net N$6: now also D5.C, R5.2; no longer J4.2, U$4.PG2
- net VBAT: now also C1.+, J9.1, J9.2, J9.3, VBAT.1, VBAT.2, VBAT.3
Other:
- moved on the sheet: BATT1, BATT3, BATT4, J4, J5

Commit message: missing part numbers
Parts:
- C1: DIST (none) -> Digikey; DISTPN (none) -> P5158-ND
- C2: DIST (none) -> Digikey; DISTPN (none) -> P5152-ND
Changed lines of the file:
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@@
 <part name="J10" library="Components" deviceset="HEADER-0.1IN-3POS" device="-FEMALE"/>
 <part name="F1" library="RemotePartsB" deviceset="SHORT" device=""/>
-<part name="C1" library="KoalaBuild" deviceset="RESOLVED-CAPACITOR-POL_" device="TH-RADIAL_ALUMINUM_18MM"/>
-<part name="C2" library="KoalaBuild" deviceset="RESOLVED-CAPACITOR-POL_" device="TH-RADIAL_ALUMINUM_6.3MM"/>
+<part name="C1" library="KoalaBuild" deviceset="RESOLVED-CAPACITOR-POL_" device="TH-RADIAL_ALUMINUM_18MM">
+<attribute name="DIST" value="Digikey"/>
+<attribute name="DISTPN" value="P5158-ND"/>
+</part>
+<part name="C2" library="KoalaBuild" deviceset="RESOLVED-CAPACITOR-POL_" device="TH-RADIAL_ALUMINUM_6.3MM">
+<attribute name="DIST" value="Digikey"/>
+<attribute name="DISTPN" value="P5152-ND"/>
+</part>
 <part name="+3V1" library="supply1" deviceset="+3V3" device=""/>
 <part name="GND3" library="supply1" deviceset="GND" device=""/>
